File: esp-switch-single-ledstrip.kicad_pcb (KiCad board)
At the start: 2 copper layers, 50 x 50 mm, 43 parts, among them J1 Conn_01x03_Socket, J2 Conn_01x05_Socket, J3 Conn_01x07_Socket, J4 Conn_01x03_Pin, Q1 TSM2302CX, Q2 TSM2302CX, Q3 TSM2302CX, Q5 BC847BS, Q6 TSM2302CX, U1 TPS54202DDC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

Commit message: Updates
Parts:
- removed R10, R15, R16, R17, R18, R8, R9: 10k, Resistor_SMD:R_0805_2012Metric_Pad1.20x1.40mm_HandSolder
- removed R11, R12, R13, R14: 10R, Resistor_SMD:R_0805_2012Metric_Pad1.20x1.40mm_HandSolder
- added C8: 100n, Capacitor_SMD:C_0805_2012Metric_Pad1.18x1.45mm_HandSolder, F.Cu at (122.2, 72.8)
- added D2: SMAJ12A, Diode_SMD:D_SMA, F.Cu at (114.4, 87.6)
- added R19: 10k, Resistor_SMD:R_0805_2012Metric_Pad1.20x1.40mm_HandSolder, F.Cu at (143.3, 77.5)
- added RN2: 10K, Resistor_SMD:R_Array_Convex_4x0612, F.Cu at (135.0, 78.0)
- added RN3: 10R, Resistor_SMD:R_Array_Convex_4x0612, F.Cu at (146.6, 77.9)
- added U3: 7408, Package_SO:TSSOP-14_4.4x5mm_P0.65mm, F.Cu at (120.7, 63.9)
- moved C6 29.0 mm to (146.0, 63.0), turned to 0 degrees
- moved R7 12.8 mm to (120.9, 55.9), turned to 0 degrees
- moved R5 4.02 mm to (145.9, 71.9)
- moved Q5 4.02 mm to (145.9, 66.2)
- moved R6 4.02 mm to (145.9, 69.3)
- moved C4 3.43 mm to (129.8, 83.9)
- moved C5 3.43 mm to (133.6, 83.9)
- moved C2 3.43 mm to (121.5, 86.5)
- moved D1 3.43 mm to (117.7, 86.5)
- moved R1 3.43 mm to (119.6, 92.2)
- moved R2 3.43 mm to (119.6, 95.4)
- moved R3 3.43 mm to (130.4, 89.5)
- moved R4 3.43 mm to (134.9, 89.0)
- moved C3 3.43 mm to (126.0, 92.8)
- moved C1 3.43 mm to (126.0, 84.6)
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Connections:
- Q1 pad 1: /GPIO13 -> Net-(Q1-G)
- Q2 pad 1: /GPIO5 -> Net-(Q2-G)
- Q3 pad 1: /GPIO12 -> Net-(Q3-G)
- Q6 pad 1: /GPIO14 -> Net-(Q6-G)
- R7 pad 1: /GPIO13 -> GND
- R7 pad 2: GND -> /DRIVE_EN
- U2 pad 16: unconnected-(U2-GPIO15-Pad16) -> Net-(U2-GPIO15)
- U2 pad 19: unconnected-(U2-GPIO4-Pad19) -> /DRIVE_EN
Routing:
- net +3V3: track 59.4 -> 13.5 mm
- net /DRIVE_EN: track 0.00 -> 37.3 mm, vias 0 -> 2
- net Net-(J3-Pin_4): track 27.3 -> 0.00 mm
- net Net-(J3-Pin_2): track 25.7 -> 0.00 mm, vias 1 -> 0
- net Net-(J3-Pin_3): track 25.7 -> 0.00 mm, vias 1 -> 0
- net Net-(J3-Pin_1): track 23.1 -> 0.00 mm
- net /RXD: track 4.94 -> 25.7 mm
- net /EN: track 19.3 -> 4.62 mm
- net GND: track 13.0 -> 0.14 mm, vias 89 -> 55
- net Net-(U2-GPIO15): track 0.00 -> 8.08 mm
- net Net-(Q2-G): track 0.00 -> 7.77 mm
- net /GPIO0: track 9.48 -> 16.5 mm
- net Net-(Q1-G): track 0.00 -> 6.85 mm
- net /GPIO2: track 3.88 -> 10.1 mm
- net Net-(Q6-G): track 0.00 -> 4.39 mm
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