File: esp-switch-single-ledstrip.kicad_sch (KiCad schematic)
At the start: 43 parts, among them J1 Conn_01x03_Socket, J2 Conn_01x05_Socket, J3 Conn_01x07_Socket, J4 Conn_01x03_Pin, Q1 TSM2302CX, Q2 TSM2302CX, Q3 TSM2302CX, Q5 BC847BS, Q6 TSM2302CX, U1 TPS54202DDC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

Commit message: Updates
Parts:
- removed R10, R15, R16, R17, R18, R8, R9: 10k, Resistor_SMD:R_0805_2012Metric_Pad1.20x1.40mm_HandSolder, symbol Device:R
- removed R11, R12, R13, R14: 10R, Resistor_SMD:R_0805_2012Metric_Pad1.20x1.40mm_HandSolder, symbol Device:R
- added C8: 100n, Capacitor_SMD:C_0805_2012Metric_Pad1.18x1.45mm_HandSolder, symbol Device:C
- added D2: SMAJ12A, Diode_SMD:D_SMA, symbol Diode:SMAJ12A
- added R19: 10k, Resistor_SMD:R_0805_2012Metric_Pad1.20x1.40mm_HandSolder, symbol Device:R
- added RN2: 10K, Resistor_SMD:R_Array_Convex_4x0612, symbol Device:R_Pack04
- added RN3: 10R, Resistor_SMD:R_Array_Convex_4x0612, symbol Device:R_Pack04_Split
- added U3: 7408, Package_SO:TSSOP-14_4.4x5mm_P0.65mm, symbol 74xx_IEEE:7408
- D1: Lomex (none) -> 83-08-27
Connections:
- net +12VA: now also D2.2 (A2)
- net +3V3: now also C8.1, RN2.1 (R1.1), RN2.2 (R2.1), RN2.3 (R3.1), RN2.4 (R4.1), U3.14 (VCC), U3.14 (VCC), U3.14 (VCC), U3.14 (VCC)
- net EN: now also RN2.8 (R1.2)
- net GND: now also R7.1, C8.2, D2.1 (A1), R19.1, U3.7 (GND), U3.7 (GND), U3.7 (GND), U3.7 (GND); no longer R7.2
- net GPIO0: now also RN2.6 (R3.2)
- net GPIO12: now also U3.9; no longer Q3.1 (G)
- net GPIO13: now also U3.13; no longer Q1.1 (G), R7.1
- net GPIO14: now also U3.5; no longer Q6.1 (G)
- net GPIO2: now also RN2.5 (R4.2)
- net GPIO5: now also U3.1; no longer Q2.1 (G)
- net RXD: now also RN3.6 (R3.2)
- net TXD: now also RN3.5 (R4.2)
- net nRST: now also RN2.7 (R2.2)
- net at U2.16 (GPIO15): now also R19.2
- net DRIVE_EN: now reaches U2.19 (GPIO4)
- net DRIVE_EN: now also R7.2, U3.10, U3.12, U3.2, U3.4
- net at J3.1 (Pin_1): now also RN3.1 (R1.1)
- net at Q5.1 (E1), R5.2: now also RN3.8 (R1.2)
- net at Q5.4 (E2), R6.2: now also RN3.7 (R2.2)
- net at J3.4 (Pin_4): now also RN3.3 (R3.1)
- net at J3.2 (Pin_2): now also RN3.2 (R2.1)
- net at J3.3 (Pin_3): now also RN3.4 (R4.1)
- new net: Q3.1 (G), U3.8
- new net: Q2.1 (G), U3.3
- new net: Q1.1 (G), U3.11
- new net: Q6.1 (G), U3.6
- no-connect marks 11 -> 9
Other:
- moved on the sheet: C6, H1, H2, H3, H4, J2, J4, Q1, Q2, Q3, Q6
